File: KiCad/Masterchefsitov1.kicad_pcb (KiCad board)
At the start: 2 copper layers, 117.5 x 87.5 mm, 15 parts, among them J1 Screw_Terminal_01x04, J2 Conn_01x07, J3 Conn_01x08, Q1 MMBT3906, U1 ESP32-DEVKIT-V1, U2 HX711

Commit message: Bloque+PCB
Parts:
- R1, R2, R3, R4, R5: footprint Resistor_SMD:R_0201_0603Metric_Pad0.64x0.40mm_HandSolder -> Resistor_SMD:R_0402_1005Metric_Pad0.72x0.64mm_HandSolder
- moved C4 8.42 mm to (126.0, 70.2)
- moved J1 4.54 mm to (99.0, 74.4)
- moved C1 3.25 mm to (119.1, 87.4)
- moved C3 2.72 mm to (110.4, 81.6), turned to 0 degrees
- moved R4 2.47 mm to (113.8, 80.6), turned to -90 degrees
- moved Q1 2.12 mm to (110.5, 75.8)
- moved U2 2.03 mm to (119.2, 81.4)
- moved C2 1.89 mm to (113.8, 82.6)
- moved R2 1.51 mm to (110.2, 86.6)
- moved R1 1.39 mm to (110.2, 84.2)
- moved R3 1.26 mm to (110.4, 80.4)
Connections:
- R5 pad 1: +3V3 -> BL_LCD
- U1 pad 10: D/C_LCD -> unconnected-(U1-Pad10)
- U1 pad 12: unconnected-(U1-Pad12) -> BL_LCD
- U1 pad 3: unconnected-(U1-Pad3) -> D/C_LCD
- U2 pad 10: GND3 -> +3V3
Routing:
- net GND3: track 86.9 -> 79.8 mm
- net Net-(J1-Pad4): track 18.2 -> 11.9 mm
- net Net-(J1-Pad3): track 16.5 -> 10.8 mm
- net +3V3: track 110.0 -> 106.2 mm
- net Net-(C1-Pad1): track 7.50 -> 11.1 mm
- net Net-(C1-Pad2): track 5.38 -> 8.92 mm
- net D/C_LCD: track 135.8 -> 133.4 mm
- net Net-(C3-Pad1): track 26.0 -> 23.8 mm
- net Net-(R3-Pad1): track 3.87 -> 6.01 mm
- net SCK_HX711: track 13.0 -> 10.9 mm
- net DT_HX711: track 12.8 -> 10.8 mm
- net Net-(Q1-Pad1): track 4.07 -> 5.76 mm
