File: KiCad/Masterchefsitov1.kicad_sch (KiCad schematic)
At the start: 1 part, among them U1 ESP32-DEVKIT-V1

Commit message: Bloque+PCB
Connections:
- net D/C_LCD: now also U1.3 (D15); no longer U1.10 (D19)
- net BL_LCD: now reaches U1.12 (RX0)
- no-connect marks 13 -> 12
Changed lines of the file:
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@@
   (no_connect (at 105.156 84.074))
   (no_connect (at 105.156 86.614))
-  (no_connect (at 105.156 89.154))
+  (no_connect (at 105.156 94.234))
   (no_connect (at 105.156 96.774))
   (no_connect (at 135.636 61.214))
-  (no_connect (at 135.636 58.674))
   (no_connect (at 105.156 51.054))
   (no_connect (at 105.156 61.214))
@@
     (stroke (width 0) (type default) (color 0 0 0 0))
   )
+  (wire (pts (xy 100.076 89.154) (xy 105.156 89.154))
+    (stroke (width 0) (type default) (color 0 0 0 0))
+  )
   (wire (pts (xy 135.636 91.694) (xy 139.954 91.694))
     (stroke (width 0) (type default) (color 0 0 0 0))
@@
     (stroke (width 0) (type default) (color 0 0 0 0))
   )
-  (wire (pts (xy 100.076 94.234) (xy 105.156 94.234))
+  (wire (pts (xy 100.076 91.694) (xy 105.156 91.694))
     (stroke (width 0) (type default) (color 0 0 0 0))
   )
-  (wire (pts (xy 100.076 91.694) (xy 105.156 91.694))
+  (wire (pts (xy 135.636 58.674) (xy 138.176 58.674))
     (stroke (width 0) (type default) (color 0 0 0 0))
   )
@@
     )
   )
-  (global_label "D{slash}C_LCD" (shape output) (at 100.076 94.234 180) (fields_autoplaced)
+  (global_label "D{slash}C_LCD" (shape output) (at 100.076 89.154 180) (fields_autoplaced)
     (effects (font (size 1.27 1.27)) (justify right))
-    (property "Intersheet References" "${INTERSHEET_REFS}" (id 0) (at 89.2567 94.1546 0)
+    (property "Intersheet References" "${INTERSHEET_REFS}" (id 0) (at 89.2567 89.0746 0)
       (effects (font (size 1.27 1.27)) (justify right) hide)
     )
   )
+  (global_label "BL_LCD" (shape output) (at 138.176 58.674 0) (fields_autoplaced)
+    (effects (font (size 1.27 1.27)) (justify left))
+    (property "Intersheet References" "${INTERSHEET_REFS}" (id 0) (at 147.4229 58.5946 0)
+      (effects (font (size 1.27 1.27)) (justify left) hide)
+    )
+  )
   (symbol (lib_id "power:GND3") (at 139.446 106.934 0) (mirror y) (unit 1)
     (in_bom yes) (on_board yes) (fields_autoplaced)
@@
       (reference "#PWR0102") (unit 1) (value "GND3") (footprint "")
     )
+    (path "/2c8304a2-f015-4f1b-9731-93bd15cb0d3a/01c1226a-87a0-4591-930b-8b2a23d3785d"
+      (reference "#PWR0103") (unit 1) (value "+3V3") (footprint "")
+    )
     (path "/2c8304a2-f015-4f1b-9731-93bd15cb0d3a/5550e554-b257-407a-b53d-85e7fe4e1668"
       (reference "C1") (unit 1) (value "0.1u") (footprint "Capacitor_SMD:C_0201_0603Metric")
@@
     )
     (path "/2c8304a2-f015-4f1b-9731-93bd15cb0d3a/8fac41ae-06a3-4a5f-9bcc-c880f2079bcb"
-      (reference "R1") (unit 1) (value "100") (footprint "Resistor_SMD:R_0201_0603Metric_Pad0.64x0.40mm_HandSolder")
+      (reference "R1") (unit 1) (value "100") (footprint "Resistor_SMD:R_0402_1005Metric")
     )
     (path "/2c8304a2-f015-4f1b-9731-93bd15cb0d3a/1a417331-cdf2-479f-8548-d02b1c4dd364"
-      (reference "R2") (unit 1) (value "100") (footprint "Resistor_SMD:R_0201_0603Metric_Pad0.64x0.40mm_HandSolder")
+      (reference "R2") (unit 1) (value "100") (footprint "Resistor_SMD:R_0402_1005Metric_Pad0.72x0.64mm_HandSolder")
     )
     (path "/2c8304a2-f015-4f1b-9731-93bd15cb0d3a/3a93cf8a-7548-4743-8fbd-e74b9849930b"
-      (reference "R3") (unit 1) (value "R") (footprint "Resistor_SMD:R_0201_0603Metric_Pad0.64x0.40mm_HandSolder")
+      (reference "R3") (unit 1) (value "R") (footprint "Resistor_SMD:R_0402_1005Metric")
     )
     (path "/2c8304a2-f015-4f1b-9731-93bd15cb0d3a/4f9c8501-ef70-491d-9c5f-8dbc23e0dcde"
-      (reference "R4") (unit 1) (value "R") (footprint "Resistor_SMD:R_0201_0603Metric_Pad0.64x0.40mm_HandSolder")
+      (reference "R4") (unit 1) (value "R") (footprint "Resistor_SMD:R_0402_1005Metric")
     )
     (path "/2c8304a2-f015-4f1b-9731-93bd15cb0d3a/620d1411-4a18-4b2c-bcc6-d2a20711d151"
-      (reference "R5") (unit 1) (value "R") (footprint "Resistor_SMD:R_0201_0603Metric_Pad0.64x0.40mm_HandSolder")
+      (reference "R5") (unit 1) (value "R") (footprint "Resistor_SMD:R_0402_1005Metric")
     )
     (path "/ef4b5fbf-a35c-4353-a03a-1b328d8c472e"
