File: KiCad/Perifericos.kicad_sch (KiCad schematic)
At the start: 14 parts, among them J2 Conn_01x07, J3 Conn_01x08

Commit message: Bloque+PCB
Parts:
- C1, C2, C3, C4: value (none) -> 0.1u; footprint (none) -> Capacitor_SMD:C_0201_0603Metric
- J1: value (none) -> Screw_Terminal_01x04; footprint (none) -> TerminalBlock:TerminalBlock_bornier-4_P5.08mm
- Q1: value (none) -> MMBT3906; footprint (none) -> Package_TO_SOT_SMD:SOT-23
- R1: value (none) -> 100; footprint (none) -> Resistor_SMD:R_0402_1005Metric
- R2: value (none) -> 100; footprint (none) -> Resistor_SMD:R_0402_1005Metric_Pad0.72x0.64mm_HandSolder
- R3, R4: value (none) -> R; footprint (none) -> Resistor_SMD:R_0402_1005Metric
- R5: footprint Resistor_SMD:R_0201_0603Metric_Pad0.64x0.40mm_HandSolder -> Resistor_SMD:R_0402_1005Metric
- U2: value (none) -> HX711; footprint (none) -> HX711:SOP127P600X180-16N
Connections:
- net +3V3: now also U2.10 (INB+); no longer R5.1
- net GND3: no longer U2.10 (INB+)
- new net BL_LCD: R5.1
Other:
- moved on the sheet: R5
